Commit message: 1
1

File: src/nova5/urdf/system/system.xacro (robot description, xacro)
@@ -6,5 +6,5 @@
         <parent link="base_frame_link"/>
         <child link="base_link"/>
-        <origin xyz="0 0 0.025" rpy="0 0 1.570796327"/>
+        <origin xyz="0 0 0.026" rpy="0 0 1.570796327"/>
     </joint>
     <link name='world' />
@@ -14,6 +14,13 @@
         <child link="base_frame_link" />
     </joint>
-    <xacro:include filename="$(find nova5)/urdf/arm/nova5_ros2_control.xacro" />
-    <xacro:nova5_robot_ros2_control name="FakeSystem"/>
+    <xacro:include filename="$(find nova5)/urdf/obstacle/box_0.xacro" />
+    <joint name="box_0_joint" type="fixed">
+        <parent link="base_link"/>
+        <child link="box_0_link"/>
+        <origin xyz="-0.5615372 -0.1361008 0.8" rpy="3.141592654 0 1.570796327"/>
+        <!-- -0.5615372 -0.1361008 0.7732302 -->
+    </joint>
+    <!-- <xacro:include filename="$(find nova5)/urdf/arm/nova5_ros2_control.xacro" />
+    <xacro:nova5_robot_ros2_control name="FakeSystem"/> -->
 <!--
     <gazebo>
