Commit message: 1
1

File: src/nova5/urdf/arm/nova5_robot.xacro (robot description, xacro)
@@ -354,5 +354,5 @@
             <origin
                 xyz="0 0 0"
-                rpy="0 0 0" />
+                rpy="0 0 -3.14159" />
             <geometry>
                 <mesh
@@ -368,5 +368,5 @@
             <origin
                 xyz="0 0 0"
-                rpy="0 0 0" />
+                rpy="0 0 -3.14159" />
             <geometry>
                 <mesh
@@ -392,2 +392,3 @@
     </joint>
 </robot>
+<!-- rpy="-1.5708 -3.14159 0" -->

File: src/nova5/urdf/system/system.xacro (robot description, xacro)
@@ -3,4 +3,20 @@
     <xacro:include filename="$(find nova5)/urdf/arm/nova5_robot.xacro" />
     <xacro:include filename="$(find nova5)/urdf/frame/door_frame.xacro" />
+    <!-- 转接板 -->
+    <xacro:include filename="$(find nova5)/urdf/gripper/adapter.xacro"/>
+    <joint name="adapter_arm_joint" type="fixed">
+        <parent link="Link6"/>
+        <child link="adapter_link"/>
+        <origin xyz="0 0 0" rpy="0 0 0"/>
+    </joint>
+    <!-- <xacro:jxs_adapter prefix="gripper_" parent="Link6"/> -->
+    <!-- 夹爪 -->
+    <xacro:include filename="$(find nova5)/urdf/gripper/RG52_050.xacro"/>
+    <joint name="gripper_base_joint" type="fixed">
+        <parent link="adapter_link"/>
+        <child link="gripper_base_link"/>
+        <origin xyz="0 0 0.0241" rpy="0 0 0"/>
+    </joint>
+    <!-- <xacro:rg52_gripper prefix="gripper_" parent="gripper_plate2"/> -->
     <joint name="arm_mount_joint" type="fixed">
         <parent link="base_frame_link"/>
@@ -14,11 +30,10 @@
         <child link="base_frame_link" />
     </joint>
-    <xacro:include filename="$(find nova5)/urdf/obstacle/box_0.xacro" />
+    <!-- <xacro:include filename="$(find nova5)/urdf/obstacle/box_0.xacro" />
     <joint name="box_0_joint" type="fixed">
         <parent link="base_link"/>
         <child link="box_0_link"/>
         <origin xyz="-0.5615372 -0.1361008 0.8" rpy="3.141592654 0 1.570796327"/>
-        <!-- -0.5615372 -0.1361008 0.7732302 -->
-    </joint>
+    </joint> -->
     <!-- <xacro:include filename="$(find nova5)/urdf/arm/nova5_ros2_control.xacro" />
     <xacro:nova5_robot_ros2_control name="FakeSystem"/> -->
