Commit message: 1
1

File: src/nova5/urdf/gripper/RG52_050.xacro (robot description, xacro)
@@ -188,4 +188,17 @@
         <mimic joint="gripper_joint_1" multiplier="1" offset="0" />
     </joint>
+    <link name="finger_tips_link">
+    </link>
+    <joint
+        name="finger_tips_joint"
+        type="fixed">
+        <origin
+            xyz="0 0 0.18750"
+            rpy="0 0 0" />
+        <parent
+            link="gripper_base_link" />
+        <child
+            link="finger_tips_link" />
+    </joint>
     <link name="grip_link">
     </link>

Commit message: 1
1

File: src/nova5/urdf/gripper/RG52_050.xacro (robot description, xacro)
@@ -34,10 +34,10 @@
         <collision>
             <origin
-                xyz="0 0 0"
-                rpy="0 0 0" />
-            <geometry>
+                xyz="0 0 0.05275"
+                rpy="0 0 0" />
+            <!-- <geometry>
                 <mesh
                 filename="package://nova5/meshes/gripper/gripper_base_link.STL" />
-            </geometry>
+            </geometry> -->
             <geometry>
                 <cylinder radius="0.0375" length="0.1055"/>

File: src/nova5/urdf/gripper/adapter.xacro (robot description, xacro)
@@ -34,4 +34,20 @@
             </geometry>
         </collision>
+        <!-- 构建夹具线区域 -->
+        <visual>
+            <origin xyz='0.0 -0.077 0.0225' rpy='0.0 0.0 0.0'/>
+            <geometry>
+                <box size="0.04 0.07 0.095"/>
+            </geometry>
+            <material name='black'>
+                <color rgba='0.0 0.0 0.0 0.5'/>
+            </material>
+        </visual>
+        <collision>
+            <origin xyz='0.0 -0.077 0.0225' rpy='0.0 0.0 0.0'/>
+            <geometry>
+                <box size="0.04 0.07 0.095"/>
+            </geometry>
+        </collision>
     </link>
 </robot>

File: src/nova5/urdf/system/system.xacro (robot description, xacro)
@@ -30,10 +30,11 @@
         <child link="base_frame_link" />
     </joint>
-    <!-- <xacro:include filename="$(find nova5)/urdf/obstacle/box_0.xacro" />
+    <xacro:include filename="$(find nova5)/urdf/obstacle/box_0.xacro" />
     <joint name="box_0_joint" type="fixed">
         <parent link="base_link"/>
         <child link="box_0_link"/>
-        <origin xyz="-0.5615372 -0.1361008 0.8" rpy="3.141592654 0 1.570796327"/>
-    </joint> -->
+        <!-- <origin xyz="0 0 0" rpy="3.141592654 0 1.570796327"/> -->
+        <origin xyz="0.449 0.019 0.985" rpy="3.126 0.002 -1.5376"/>
+    </joint>
     <!-- <xacro:include filename="$(find nova5)/urdf/arm/nova5_ros2_control.xacro" />
     <xacro:nova5_robot_ros2_control name="FakeSystem"/> -->
